File: Electrical/KiCad/Gun board/Gun board.sch (KiCad schematic (older format))
At the start: 58 parts

Commit message: Finished V1 of schematic
Parts:
- added C?: CP, symbol Device:CP
- added C?: C, symbol Device:C
- added J?: Micro_SD_Card, symbol Connector:Micro_SD_Card
- added LS?: Speaker, symbol Device:Speaker
- added Q? (x2): 2N3904, Package_TO_SOT_THT:TO-92_Inline, symbol Transistor_BJT:2N3904
- added R? (x4): R, symbol Device:R
- added R? (x2): 4.7kΩ, symbol Device:R_Small
- added R?: 10Ω, symbol Device:R
- added U?: LM386, symbol Amplifier_Audio:LM386
- added U?: MCP4018, symbol custom_components:MCP4018
Connections:
- net +3V3: now also U?.3 (VDD), U?.6 (A0), J?.4 (VDD), Q?.3 (C), R?.1, R?.1, R?.1, U?.1 (VDD)
- net +5V: now also U?.6 (V+)
- net CE: now also R?.2, R?.2; no longer U?.3 (CE)
- net GND: now also U?.2 (VSS), J?.6 (VSS), J?.9 (SHIELD), LS?.2, Q?.1 (E), R?.2, R?.2, U?.2 (-), U?.2 (VSS), U?.4 (GND)
- net I2C_SCL: now also U?.5 (SCL), R?.2, U?.3 (SCL)
- net I2C_SDA: now also U?.4 (SDA), R?.2, U?.4 (SDA)
- net MISO: now also J?.7 (DAT0)
- net MOSI: now also J?.3 (CMD)
- net SCK: now also J?.5 (CLK)
- net SPK: now reaches U?.1 (VOUT)
- net SPK: now also U?.6 (A)
- new net: Q?.2 (B), R?.1 (x2)
- new net: U?.3 (+), U?.5 (W)
- new net: C?.1, C?.1, U?.5
- new net: C?.2, LS?.1
- new net: C?.2, R?.1
- new net CE0: Q?.3 (C), R?.2, U?.3 (CE)
- new net CE1: J?.2 (DAT3/CD), Q?.1 (E), R?.1
- no-connect marks 1 -> 6
Other:
- note added: "3.3V POWER SUPPLY"
- note added: "5V POWER SUPPLY"
- note added: "DECOUPLING CAPACITORS"
- note added: "DIGITAL TO ANAL LOG CONVORTER"
- note added: "LASER DIODE ARRAY"
- note added: "LASER POWER SUPPLY"
- note added: "MICOCONTROLER"
- note added: "RADIO SIGNAL TO CONNECT GUNS"
- note added: "SOUND"
- note added: "SOUND FILES/EXTRA STORAGE"
- note added: "SPI SWITCH"
- note removed: "Laser Diode Array"
- moved on the sheet: C?, R?, U?
